File: schematics/Clock3D/Clock3D.kicad_sch (KiCad schematic)
At the start: 20 parts, among them Q1 2N7000, Q2 2N7000, Q3 2N7000, Q4 2N7000, Q5 2N2222, U1 ESP-01, U2 74HC595, U3 74HC595, U4 MAN74A, U5 MAN74A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

Commit message: fix: updated schematics
Parts:
- R4: value 82 -> 220
- R5: value 22 -> 10
Connections:
- net +3V3: no longer U2.10 (~{SRCLR}), U2.16 (VCC), U3.10 (~{SRCLR}), U3.16 (VCC)
- net +5V: now also U2.10 (~{SRCLR}), U2.16 (VCC), U3.10 (~{SRCLR}), U3.16 (VCC)
Changed lines of the file:
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@@
     )
+  )
+  (symbol (lib_id "power:+5V") (at 186.055 43.815 90) (unit 1)
+    (in_bom yes) (on_board yes) (fields_autoplaced)
+    (property "Reference" "#PWR?" (id 0) (at 189.865 43.815 0)
+      (effects (font (size 1.27 1.27)) hide)
+    )
+    (property "Value" "+5V" (id 1) (at 182.88 43.8149 90)
+      (effects (font (size 1.27 1.27)) (justify left))
+    )
+    (property "Footprint" "" (id 2) (at 186.055 43.815 0)
+      (effects (font (size 1.27 1.27)) hide)
+    )
+    (property "Datasheet" "" (id 3) (at 186.055 43.815 0)
+      (effects (font (size 1.27 1.27)) hide)
+    )
+    (pin "1")
   )
   (symbol (lib_id "power:GND") (at 215.9 149.225 0) (unit 1)
@@
     (pin "1")
     (pin "2")
+  )
+  (symbol (lib_id "power:+5V") (at 196.215 80.645 0) (unit 1)
+    (in_bom yes) (on_board yes)
+    (property "Reference" "#PWR?" (id 0) (at 196.215 84.455 0)
+      (effects (font (size 1.27 1.27)) hide)
+    )
+    (property "Value" "+5V" (id 1) (at 196.215 76.2 0))
+    (property "Footprint" "" (id 2) (at 196.215 80.645 0)
+      (effects (font (size 1.27 1.27)) hide)
+    )
+    (property "Datasheet" "" (id 3) (at 196.215 80.645 0)
+      (effects (font (size 1.27 1.27)) hide)
+    )
+    (pin "1")
   )
   (symbol (lib_id "74xx:74HC595") (at 196.215 46.355 0) (unit 1)
@@
     (pin "2")
   )
-  (symbol (lib_id "power:+3.3V") (at 186.055 43.815 90) (unit 1)
-    (in_bom yes) (on_board yes) (fields_autoplaced)
-    (property "Reference" "#PWR09" (id 0) (at 189.865 43.815 0)
-      (effects (font (size 1.27 1.27)) hide)
-    )
-    (property "Value" "+3.3V" (id 1) (at 182.88 43.8149 90)
-      (effects (font (size 1.27 1.27)) (justify left))
-    )
-    (property "Footprint" "" (id 2) (at 186.055 43.815 0)
-      (effects (font (size 1.27 1.27)) hide)
-    )
-    (property "Datasheet" "" (id 3) (at 186.055 43.815 0)
-      (effects (font (size 1.27 1.27)) hide)
-    )
-    (pin "1")
-  )
-  (symbol (lib_id "power:+3.3V") (at 196.215 80.645 0) (unit 1)
-    (in_bom yes) (on_board yes) (fields_autoplaced)
-    (property "Reference" "#PWR014" (id 0) (at 196.215 84.455 0)
-      (effects (font (size 1.27 1.27)) hide)
-    )
-    (property "Value" "+3.3V" (id 1) (at 196.215 75.565 0))
-    (property "Footprint" "" (id 2) (at 196.215 80.645 0)
-      (effects (font (size 1.27 1.27)) hide)
-    )
-    (property "Datasheet" "" (id 3) (at 196.215 80.645 0)
-      (effects (font (size 1.27 1.27)) hide)
-    )
-    (pin "1")
-  )
   (symbol (lib_id "power:+3.3V") (at 54.61 43.815 90) (unit 1)
     (in_bom yes) (on_board yes) (fields_autoplaced)
@@
       (effects (font (size 1.27 1.27)) (justify left))
     )
-    (property "Value" "22" (id 1) (at 217.805 146.6849 0)
+    (property "Value" "10" (id 1) (at 217.805 146.6849 0)
       (effects (font (size 1.27 1.27)) (justify left))
     )
@@
       (effects (font (size 1.27 1.27)) (justify left))
     )
-    (property "Value" "82" (id 1) (at 198.12 146.6849 0)
+    (property "Value" "220" (id 1) (at 198.12 146.6849 0)
       (effects (font (size 1.27 1.27)) (justify left))
     )
@@
     (pin "1")
   )
-  (symbol (lib_id "power:+3.3V") (at 186.055 93.345 90) (unit 1)
-    (in_bom yes) (on_board yes) (fields_autoplaced)
-    (property "Reference" "#PWR010" (id 0) (at 189.865 93.345 0)
-      (effects (font (size 1.27 1.27)) hide)
-    )
-    (property "Value" "+3.3V" (id 1) (at 182.88 93.3449 90)
+  (symbol (lib_id "power:+5V") (at 186.055 93.345 90) (unit 1)
+    (in_bom yes) (on_board yes) (fields_autoplaced)
+    (property "Reference" "#PWR?" (id 0) (at 189.865 93.345 0)
+      (effects (font (size 1.27 1.27)) hide)
+    )
+    (property "Value" "+5V" (id 1) (at 182.88 93.3449 90)
       (effects (font (size 1.27 1.27)) (justify left))
     )
@@
     )
     (property "Datasheet" "" (id 3) (at 54.61 38.735 0)
+      (effects (font (size 1.27 1.27)) hide)
+    )
+    (pin "1")
+  )
+  (symbol (lib_id "power:+5V") (at 196.215 31.115 0) (unit 1)
+    (in_bom yes) (on_board yes)
+    (property "Reference" "#PWR?" (id 0) (at 196.215 34.925 0)
+      (effects (font (size 1.27 1.27)) hide)
+    )
+    (property "Value" "+5V" (id 1) (at 196.215 26.67 0))
+    (property "Footprint" "" (id 2) (at 196.215 31.115 0)
+      (effects (font (size 1.27 1.27)) hide)
+    )
+    (property "Datasheet" "" (id 3) (at 196.215 31.115 0)
       (effects (font (size 1.27 1.27)) hide)
     )
@@
     (pin "9")
   )
-  (symbol (lib_id "power:+3.3V") (at 196.215 31.115 0) (unit 1)
-    (in_bom yes) (on_board yes) (fields_autoplaced)
-    (property "Reference" "#PWR012" (id 0) (at 196.215 34.925 0)
-      (effects (font (size 1.27 1.27)) hide)
-    )
-    (property "Value" "+3.3V" (id 1) (at 196.215 25.4 0))
-    (property "Footprint" "" (id 2) (at 196.215 31.115 0)
-      (effects (font (size 1.27 1.27)) hide)
-    )
-    (property "Datasheet" "" (id 3) (at 196.215 31.115 0)
-      (effects (font (size 1.27 1.27)) hide)
-    )
-    (pin "1")
-  )
   (symbol (lib_id "power:+3.3V") (at 114.3 26.035 0) (unit 1)
     (in_bom yes) (on_board yes) (fields_autoplaced)
@@
       (reference "#PWR08") (unit 1) (value "+3.3V") (footprint "")
     )
-    (path "/48ce1cb4-bc17-45c1-bbe9-296fc0376f0c"
-      (reference "#PWR09") (unit 1) (value "+3.3V") (footprint "")
-    )
-    (path "/b116d6ff-2518-41b2-a506-8d0942d4bcce"
-      (reference "#PWR010") (unit 1) (value "+3.3V") (footprint "")
-    )
     (path "/af36458b-699e-4396-9fdc-bf0a08486fb1"
       (reference "#PWR011") (unit 1) (value "GND") (footprint "")
     )
-    (path "/ec32f443-c77a-45cd-865c-5ff21dcb02fc"
-      (reference "#PWR012") (unit 1) (value "+3.3V") (footprint "")
-    )
     (path "/747b34b1-e4eb-49d0-be55-440c40c6848d"
       (reference "#PWR013") (unit 1) (value "GND") (footprint "")
     )
-    (path "/52faed5d-3121-4c47-aeec-123556c517fe"
-      (reference "#PWR014") (unit 1) (value "+3.3V") (footprint "")
-    )
     (path "/9c82765b-aaa8-4199-afdc-6c04806fee1a"
       (reference "#PWR015") (unit 1) (value "GND") (footprint "")
@@
       (reference "#PWR017") (unit 1) (value "GND") (footprint "")
     )
+    (path "/05b89307-98f9-4bfc-af82-e6d88b5d3895"
+      (reference "#PWR?") (unit 1) (value "+5V") (footprint "")
+    )
+    (path "/33594c17-d11f-4ce8-ae97-9aacdd2e7d5c"
+      (reference "#PWR?") (unit 1) (value "+5V") (footprint "")
+    )
+    (path "/b1c36f6e-75a8-4c4c-8ed4-d43e9de62446"
+      (reference "#PWR?") (unit 1) (value "+5V") (footprint "")
+    )
+    (path "/e65e60e0-c00d-4661-9543-ef9ae9cb521a"
+      (reference "#PWR?") (unit 1) (value "+5V") (footprint "")
+    )
     (path "/2ae03dc0-9fea-4c5e-bbaf-0b1a865d7166"
       (reference "D1") (unit 1) (value "LED") (footprint "")
@@
     )
     (path "/a8eb2624-35c6-43d8-bdb5-f041ba5bf5ab"
-      (reference "R4") (unit 1) (value "82") (footprint "")
+      (reference "R4") (unit 1) (value "220") (footprint "")
     )
     (path "/6e9e5f83-db49-4e84-893d-cfd7e6370871"
-      (reference "R5") (unit 1) (value "22") (footprint "")
+      (reference "R5") (unit 1) (value "10") (footprint "")
     )
     (path "/e02d1a75-0fa2-415c-adae-a5074fe3e755"
